Commit message: asus_xtion_pro URDF: Use same tfs as openni2_launch

File: lucia_turtlebot_description/urdf/sensors/asus_xtion_pro.urdf.xacro (robot description, xacro)
@@ -5,11 +5,35 @@
   <xacro:property name="M_SCALE" value="0.001"/>
   <!-- <xacro:property name="asus_xtion_pro_cam_py" value="0.0205"/> -->
-  <xacro:property name="asus_xtion_pro_depth_rel_rgb_py" value="0.0270" />
-  <xacro:property name="asus_xtion_pro_cam_rel_rgb_py"   value="-0.0220" />
   <xacro:macro name="sensor_asus_xtion_pro" params="parent top_cam_px top_cam_py top_cam_pz top_cam_or top_cam_op top_cam_oy">
-    <joint name="top_camera_rgb_joint" type="fixed">
+    <joint name="top_camera_joint" type="fixed">
       <origin xyz="${top_cam_px} ${top_cam_py} ${top_cam_pz}"
               rpy="${top_cam_or} ${top_cam_op} ${top_cam_oy}"/>
       <parent link="${parent}"/>
+      <child link="top_camera_link"/>
+    </joint>
+    <link name="top_camera_link">
+      <visual>
+        <origin xyz="-0.01 -0.068 0" rpy="${-M_PI/2} -${M_PI} ${-M_PI/2}"/>
+        <geometry>
+          <mesh filename="package://turtlebot_description/meshes/sensors/asus_xtion_pro_live.dae" scale="${M_SCALE} ${M_SCALE} ${M_SCALE}"/>
+        </geometry>
+      </visual>
+      <collision>
+        <origin xyz="0 -0.068 0" />
+        <geometry>
+        <box size="0.0730 0.2760 0.0720"/>
+      </geometry>
+      </collision>
+      <inertial>
+        <mass value="0.170" />
+        <origin xyz="0 -0.068 0" />
+        <inertia ixx="0.001152600" ixy="0.0" ixz="0.0"
+                 iyy="0.000148934" iyz="0.0"
+                 izz="0.001154654" />
+      </inertial>
+    </link>
+    <joint name="top_camera_rgb_joint" type="fixed">
+      <origin xyz="0 -0.045 0" rpy="0 0 0" />
+      <parent link="top_camera_link"/>
       <child link="top_camera_rgb_frame" />
     </joint>
@@ -21,34 +45,7 @@
     </joint>
     <link name="top_camera_rgb_optical_frame"/>
-    <joint name="top_camera_joint" type="fixed">
-      <origin xyz="0 ${asus_xtion_pro_cam_rel_rgb_py} 0"
-              rpy="0 0 0"/>
-      <parent link="top_camera_rgb_frame"/>
-      <child link="top_camera_link"/>
-    </joint>
-    <link name="top_camera_link">
-      <visual>
-        <origin xyz="-0.01 0 0" rpy="${-M_PI/2} -${M_PI} ${-M_PI/2}"/>
-        <geometry>
-          <mesh filename="package://turtlebot_description/meshes/sensors/asus_xtion_pro_live.dae" scale="${M_SCALE} ${M_SCALE} ${M_SCALE}"/>
-        </geometry>
-      </visual>
-      <collision>
-        <origin xyz="0.0 0.0 0.0" rpy="0 0 0" />
-        <geometry>
-        <box size="0.0730 0.2760 0.0720"/>
-      </geometry>
-      </collision>
-      <inertial>
-        <mass value="0.170" />
-        <origin xyz="0 0 0" />
-        <inertia ixx="0.001152600" ixy="0.0" ixz="0.0"
-                 iyy="0.000148934" iyz="0.0"
-                 izz="0.001154654" />
-      </inertial>
-    </link>
     <joint name="top_camera_depth_joint" type="fixed">
-      <origin xyz="0 ${asus_xtion_pro_depth_rel_rgb_py} 0" rpy="0 0 0" />
-      <parent link="top_camera_rgb_frame" />
+      <origin xyz="0 -0.02 0" rpy="0 0 0" />
+      <parent link="top_camera_link"/>
       <child link="top_camera_depth_frame" />
     </joint>
